File: Transformer Less Power supply/pcb/Transformer Less Power supply.kicad_sch (KiCad schematic)
At the start: 0 parts

Commit message: Servo Tester and Ac to DC Power Supply without Transformer added
Parts:
- added C1: 0.1uF, Capacitor_THT:C_Disc_D4.7mm_W2.5mm_P5.00mm, symbol Device:C
- added C2: 1000uF, Capacitor_THT:CP_Radial_D10.0mm_P5.00mm, symbol Device:C_Polarized_US
- added C3: 470uF, Capacitor_THT:CP_Radial_D10.0mm_P3.80mm, symbol Device:C_Polarized_US
- added C4: 225k/2.2uF, Capacitor_THT:C_Rect_L13.5mm_W5.0mm_P10.00mm_FKS3_FKP3_MKS4, symbol Device:C
- added D1, D2, D3, D4: 1N4007, Diode_THT:D_DO-41_SOD81_P10.16mm_Horizontal, symbol Diode:1N4007
- added D5, D6: D_Zener, Diode_THT:D_A-405_P7.62mm_Horizontal, symbol Device:D_Zener
- added D7: LED, LED_THT:LED_D5.0mm, symbol Device:LED
- added J1, J2: Screw_Terminal_01x02, TerminalBlock:TerminalBlock_bornier-2_P5.08mm, symbol Connector:Screw_Terminal_01x02
- added R1: 1M, Resistor_THT:R_Axial_DIN0207_L6.3mm_D2.5mm_P7.62mm_Horizontal, symbol Device:R
- added R2, R3: 20k, Resistor_THT:R_Axial_DIN0207_L6.3mm_D2.5mm_P7.62mm_Horizontal, symbol Device:R
- added R4: 2.2k, Resistor_THT:R_Axial_DIN0207_L6.3mm_D2.5mm_P7.62mm_Horizontal, symbol Device:R
- added U1: LM7805_TO220, Package_TO_SOT_THT:TO-220-3_Vertical, symbol Regulator_Linear:LM7805_TO220
Connections:
- new net: C1.2, C2.1, D1.1 (K), D3.1 (K), D5.1 (K), D6.1 (K), R4.2, U1.1 (VI)
- new net: D3.2 (A), D4.1 (K), J1.1 (Pin_1)
- new net: C4.1, J1.2 (Pin_2), R1.1
- new net: C4.2, D1.2 (A), D2.1 (K), R1.2
- new net: D5.2 (A), R2.2
- new net: D6.2 (A), R3.2
- new net: D7.2 (A), R4.1
- new net 5V: C3.1, J2.2 (Pin_2), U1.3 (VO)
- new net GND: C1.1, C2.2, C3.2, D2.2 (A), D4.2 (A), D7.1 (K), J2.1 (Pin_1), R2.1, R3.1, U1.2 (GND)
Other:
- note added: "Transformerless Ac to Dc Power Supply"
- company: (none) -> Girish Kotalwar
- title: (none) -> Tranformerless Ac to Dc Power Supply
