File: Servo Tester/pcb/Servo Tester/Servo Tester.kicad_sch (KiCad schematic)
At the start: 10 parts, among them J1 Conn_01x02_Pin, J2 Conn_01x03_Pin, U1 NA555P

Commit message: Updated files
Other:
- note added: "Servo Tester using 555 Timer IC"
Changed lines of the file:
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@@
 		(company "Girish Kotalwar")
+	)
+	(rectangle
+		(start 74.93 58.42)
+		(end 218.44 135.89)
+		(stroke
+			(width 0)
+			(type default)
+		)
+		(fill
+			(type none)
+		)
 	)
 	(text "servo motor"
@@
 			(font
 				(size 1.27 1.27)
+			)
+		)
+	)
+	(text "Servo Tester using 555 Timer IC"
+		(exclude_from_sim no)
+		(at 116.84 64.77 0)
+		(effects
+			(font
+				(face "Bahnschrift")
+				(size 3.81 3.81)
+				(bold yes)
 			)
 		)
@@
 		)
 		(property "Value" "Conn_01x03_Pin"
-			(at 208.28 97.7899 0)
+			(at 212.09 100.33 90)
 			(effects
 				(font
@@
 		(on_board yes)
 		(dnp no)
-		(fields_autoplaced yes)
 		(property "Reference" "J1"
 			(at 85.725 86.36 0)
@@
 		)
 		(property "Value" "Conn_01x02_Pin"
-			(at 85.725 88.9 0)
-			(effects
-				(font
+			(at 81.28 86.36 90)
+			(effects
+				(font
